Commit message: Added base_footprint link in robot_core.xacro

File: dev_ws/src/burgerbot_rev1/urdf/robot_core.xacro (robot description, xacro)
@@ -6,4 +6,12 @@
     <!-- BASE LINK -->
     <link name="base_link">
+    </link>
+    <!-- BASE FOOTPRINT LINK-->
+    <joint name="base_footprint_joint" type="fixed">
+        <parent link="base_link"/>
+        <child link="base_footprint"/>
+        <origin xyz="0 0 0" rpy="0 0 0"/>
+    </joint>
+    <link name="base_footprint">
     </link>
     <!--CHASSIS LINK    (check the joint & link origin after adding wheels) -->

Commit message: Fixed the robot XACRO file

File: dev_ws/src/burgerbot_rev1/urdf/robot_core.xacro (robot description, xacro)
@@ -4,7 +4,9 @@
     <xacro:include filename="robot_dimensions.xacro" />
     <xacro:include filename="lidar.xacro" />
+    <xacro:include filename="interia_macro.xacro"/>
+    <xacro:include filename="gazebo_control.xacro"/>
     <!-- BASE LINK -->
-    <link name="base_link">
-    </link>
+    <link name="base_footprint"/>
+    <link name="base_link"/>
     <!-- BASE FOOTPRINT LINK-->
     <joint name="base_footprint_joint" type="fixed">
@@ -13,11 +15,9 @@
         <origin xyz="0 0 0" rpy="0 0 0"/>
     </joint>
-    <link name="base_footprint">
-    </link>
     <!--CHASSIS LINK    (check the joint & link origin after adding wheels) -->
     <joint name="chassis_joint" type="fixed">
         <parent link="base_link"/>
         <child link="chassis_link"/>
-        <origin xyz="0 0 0"/>
+        <origin xyz="0 0 ${wheel_radius / 2.0}"/>
     </joint>
     <link name="chassis_link">
@@ -35,10 +35,16 @@
             </geometry>
         </collision>
+        <xacro:inertial_box mass="0.5" x="${body_radius}" y="${body_radius}" z="${body_length}">
+            <origin xyz="${body_radius/2} 0 ${body_length/2}" rpy="0 0 0"/>
+        </xacro:inertial_box>
     </link>
+    <gazebo reference="chassis">
+        <material>Gazebo/Orange</material>
+    </gazebo>
     <!-- LEFT WHEEL LINK -->
     <joint name="left_wheel_joint" type="continuous">
         <parent link="base_link"/>
         <child link="left_wheel"/>
-        <origin xyz="0 0.07 0" rpy="-${pi/2} 0 0"/>
+        <origin xyz="0 0.07 ${wheel_radius}" rpy="-${pi/2} 0 0"/>
         <axis xyz="0 0 1"/>
     </joint>
@@ -46,5 +52,5 @@
         <visual>
             <geometry>
-                <cylinder radius="${wheel_radius}" length="0.02"/> <!-- 1cm thickness -->
+                <cylinder radius="${wheel_radius}" length="${wheel_thickness}"/>
             </geometry>
             <material name="white"/>
@@ -52,13 +58,19 @@
         <collision>
             <geometry>
-                <cylinder radius="${wheel_radius}" length="0.02"/> <!-- 1cm thickness -->
+                <cylinder radius="${wheel_radius}" length="${wheel_thickness}"/> <!-- 1cm thickness -->
             </geometry>
         </collision>
+        <xacro:inertial_cylinder mass="${wheel_mass}" length="${wheel_thickness}" radius="${wheel_radius}">
+            <origin xyz="0 0 0" rpy="0 0 0"/>
+        </xacro:inertial_cylinder>
     </link>
+    <gazebo reference="left_wheel">
+        <material>Gazebo/Blue</material>
+    </gazebo>
     <!-- RIGHT WHEEL LINK -->
     <joint name="right_wheel_joint" type="continuous">
         <parent link="base_link"/>
         <child link="right_wheel"/>
-        <origin xyz="0 -0.07 0" rpy="${pi/2} 0 0"/>
+        <origin xyz="0 -0.07 ${wheel_radius}" rpy="${pi/2} 0 0"/>
         <axis xyz="0 0 -1"/>
     </joint>
@@ -75,5 +87,11 @@
             </geometry>
         </collision>
+        <xacro:inertial_cylinder mass="${wheel_mass}" length="${wheel_thickness}" radius="${wheel_radius}">
+            <origin xyz="0 0 0" rpy="0 0 0"/>
+        </xacro:inertial_cylinder>
     </link>
+    <gazebo reference="right_wheel">
+        <material>Gazebo/Blue</material>
+    </gazebo>
     <!-- CASTER WHEEL LINK -->
     <joint name="caster_wheel_joint" type="fixed">
@@ -94,4 +112,12 @@
             </geometry>
         </collision>
+        <xacro:inertial_sphere mass="${caster_wheel_mass}" radius="${caster_radius}">
+            <origin xyz="0 0 0" rpy="0 0 0"/>
+        </xacro:inertial_sphere>
     </link>
+    <gazebo reference="caster_wheel">
+        <material>Gazebo/Blue</material>
+        <mu1 value="0.001"/>
+        <mu2 value="0.001"/>
+    </gazebo>
 </robot>

File: dev_ws/src/burgerbot_rev1/urdf/robot_dimensions.xacro (robot description, xacro)
@@ -5,5 +5,5 @@
   <xacro:property name="body_diameter" value="0.12"/>
   <xacro:property name="body_length" value="0.08"/>
-  <xacro:property name="body_radius" value="0.06"/>
+  <xacro:property name="body_radius" value="${body_diameter / 2.0}"/>
   <!-- Wheel dimensions -->
   <!-- Wheel diameter = 60mm (0.06 m); radius is half of that -->
@@ -12,6 +12,9 @@
   <!-- Distance between the centers of the left and right wheels = 150mm (0.15 m) -->
   <xacro:property name="wheel_separation" value="0.15"/>
-  <!-- If wheels need a small offset along x-axis, set here (0 if none) -->
-  <xacro:property name="wheel_x_offset" value="0.0"/>
+  <xacro:property name="wheel_mass" value="0.05"/>
+  <xacro:property name="wheel_thickness" value="0.026"/>
+  <xacro:property name="wheel_offset_x" value="0.226"/>
+  <xacro:property name="wheel_offset_y" value="0.1485"/>
+  <xacro:property name="wheel_offset_z" value="0.01"/>
   <!-- Lidar dimensions -->
   <!-- Represent the lidar as a cylinder with diameter = 70mm (0.07 m) -->
@@ -22,7 +25,9 @@
   <xacro:property name="lidar_offset_from_top" value="0.03"/>
   <!-- Caster wheel dimensions -->
-  <!-- Place the caster wheel at 75mm (0.075 m) from the robot center -->
   <xacro:property name="caster_distance" value="0.03"/>
-  <!-- Represent the caster as a sphere; choose a radius (e.g., 20mm or 0.02 m) -->
-  <xacro:property name="caster_radius" value="0.03"/>
+  <!-- caster_wheel_radius changed to caster_radius-->
+  <xacro:property name="caster_radius" value="0.015"/>
+  <xacro:property name="caster_wheel_mass" value="0.01"/>
+  <xacro:property name="caster_wheel_offset_x" value="0.075"/>
+    <xacro:property name="caster_wheel_offset_z" value="${wheel_offset_z - wheel_radius + caster_radius}"/>
 </robot>
